File: ESP12_Dev.sch (EAGLE design)
At the start: 10 parts

Commit message: Version one
Connections:
- removed net GPIO15: ESP_12.GPIO15, JP2.2
- net GND: now also ESP_12.GPIO15, JP2.2
Changed lines of the file:
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@@
 <pinref part="JP2" gate="G$1" pin="1"/>
 <pinref part="ESP_12" gate="G$1" pin="GND"/>
-<wire x1="73.66" y1="50.8" x2="78.74" y2="50.8" width="0.1524" layer="91"/>
+<wire x1="73.66" y1="50.8" x2="76.2" y2="50.8" width="0.1524" layer="91"/>
+<wire x1="76.2" y1="50.8" x2="78.74" y2="50.8" width="0.1524" layer="91"/>
 <wire x1="78.74" y1="50.8" x2="86.36" y2="50.8" width="0.1524" layer="91"/>
 <wire x1="78.74" y1="43.18" x2="78.74" y2="50.8" width="0.1524" layer="91"/>
 <junction x="78.74" y="50.8"/>
 <pinref part="GND1" gate="1" pin="GND"/>
+<pinref part="JP2" gate="G$1" pin="2"/>
+<pinref part="ESP_12" gate="G$1" pin="GPIO15"/>
+<wire x1="73.66" y1="53.34" x2="76.2" y2="53.34" width="0.1524" layer="91"/>
+<wire x1="76.2" y1="53.34" x2="86.36" y2="53.34" width="0.1524" layer="91"/>
+<wire x1="76.2" y1="53.34" x2="76.2" y2="50.8" width="0.1524" layer="91"/>
+<junction x="76.2" y="53.34"/>
+<junction x="76.2" y="50.8"/>
 </segment>
 <segment>
@@
 </segment>
 </net>
-<net name="GPIO15" class="0">
-<segment>
-<pinref part="ESP_12" gate="G$1" pin="GPIO15"/>
-<pinref part="JP2" gate="G$1" pin="2"/>
-<wire x1="73.66" y1="53.34" x2="86.36" y2="53.34" width="0.1524" layer="91"/>
-</segment>
-</net>
